File: BUCK_BOOST_42W.kicad_sch (KiCad schematic)
At the start: 55 parts, among them J1 Conn_01x08_Pin, J13 Conn_01x12_Socket, J14 Conn_01x16_Socket, J15 Conn_01x02_Pin, J16 Conn_01x02_Pin, J17 Conn_01x02_Pin, J2 Conn_01x03_Pin, U1 INA226, U2 INA226, U3 INA226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

Commit message: sense resistor partial changes
Other:
- added sheet Inrush_limiter (Inrush_limiter.kicad_sch)
Changed lines of the file:
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@@
+	)
+	(sheet
+		(at 175.26 90.17)
+		(size 12.7 11.43)
+		(exclude_from_sim no)
+		(in_bom yes)
+		(on_board yes)
+		(dnp no)
+		(fields_autoplaced yes)
+		(stroke
+			(width 0.1524)
+			(type solid)
+		)
+		(fill
+			(color 0 0 0 0.0000)
+		)
+		(property "Sheetname" "Inrush_limiter"
+			(at 175.26 89.4584 0)
+			(effects
+				(font
+					(size 1.27 1.27)
+				)
+				(justify left bottom)
+			)
+		)
+		(property "Sheetfile" "Inrush_limiter.kicad_sch"
+			(at 175.26 102.1846 0)
+			(effects
+				(font
+					(size 1.27 1.27)
+				)
+				(justify left top)
+			)
+		)
+		(instances
+			(project "BUCK_BOOST_42W"
+				(path "/c2919a84-19be-47b1-b680-01ad760017c4"
+					(page "14")
+				)
+			)
+		)
 	)
 	(sheet
