File: bb42.kicad_sch (KiCad schematic)
At the start: 90 parts, among them Q1 BSC0902NSI, Q2 BSC0902NSI, Q3 BSC0902NSI, Q4 BSC0902NSI, Q5 2N3904, U5 LM5176RHF

Commit message: sense resistor partial changes
Connections:
- net Vshunt+: now reaches Q2.1 (S), Q2.2 (S), Q2.3 (S), Q4.1 (S), Q4.2 (S), Q4.3 (S), R20.2, R22.1, R23.1, TP40.1
Changed lines of the file:
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@@
 	(generator "eeschema")
 	(generator_version "9.0")
-	(paper "A2")
+	(paper "A4")
 	(junction
 		(at 67.31 44.45)
@@
 		(effects
 			(font
+				(size 1.27 1.27)
+			)
+			(justify left bottom)
+		)
+	)
+	(label "Vshunt+"
+		(at 274.32 104.14 0)
+		(effects
+			(font
